File: lm5116_synchronous_buck.kicad_sch (KiCad schematic)
At the start: 65 parts, among them J10 Conn_01x01_Male, J11 Conn_01x01_Male, J12 Conn_01x01_Male, J7 Conn_01x03_Male, J8 Conn_01x01_Male, J9 Conn_01x01_Male, Q1 BSC118N10NSG, Q2 BSC118N10NSG, Q3 AO3409, U7 LM5116, U8 STUSB4700

Commit message: ERC Check Finish
Parts:
- gave numbers to parts that had none: 6
Changed lines of the file:
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@@
   (symbol (lib_id "Device:C") (at 294.64 82.55 0) (unit 1)
     (in_bom yes) (on_board yes)
-    (property "Reference" "C?" (id 0) (at 293.37 85.09 90))
+    (property "Reference" "C55" (id 0) (at 293.37 85.09 90))
     (property "Value" "100p" (id 1) (at 293.37 78.105 90))
     (property "Footprint" "Capacitor_SMD:C_0603_1608Metric" (id 2) (at 295.6052 86.36 0)
@@
   (symbol (lib_id "Transistor_FET:AO3401A") (at 283.21 158.75 270) (mirror x) (unit 1)
     (in_bom yes) (on_board yes) (fields_autoplaced)
-    (property "Reference" "Q?" (id 0) (at 283.21 148.59 90))
+    (property "Reference" "Q5" (id 0) (at 283.21 148.59 90))
     (property "Value" "AO3401A" (id 1) (at 283.21 151.13 90))
     (property "Footprint" "Package_TO_SOT_SMD:SOT-23" (id 2) (at 281.305 153.67 0)
@@
   (symbol (lib_id "Device:C_Small") (at 312.42 168.91 180) (unit 1)
     (in_bom yes) (on_board yes) (fields_autoplaced)
-    (property "Reference" "C?" (id 0) (at 314.96 167.6335 0)
+    (property "Reference" "C56" (id 0) (at 314.96 167.6335 0)
       (effects (font (size 1.27 1.27)) (justify right))
     )
@@
   (symbol (lib_id "Transistor_FET:AO3401A") (at 256.54 158.75 90) (unit 1)
     (in_bom yes) (on_board yes) (fields_autoplaced)
-    (property "Reference" "Q?" (id 0) (at 256.54 148.59 90))
+    (property "Reference" "Q4" (id 0) (at 256.54 148.59 90))
     (property "Value" "AO3401A" (id 1) (at 256.54 151.13 90))
     (property "Footprint" "Package_TO_SOT_SMD:SOT-23" (id 2) (at 258.445 153.67 0)
@@
   (symbol (lib_id "Device:R") (at 246.38 180.34 180) (unit 1)
     (in_bom yes) (on_board yes)
-    (property "Reference" "R?" (id 0) (at 243.84 180.34 90))
+    (property "Reference" "R24" (id 0) (at 243.84 180.34 90))
     (property "Value" "10k" (id 1) (at 248.92 180.34 90))
     (property "Footprint" "Resistor_SMD:R_0603_1608Metric" (id 2) (at 248.158 180.34 90)
@@
   (symbol (lib_id "Connector:Conn_01x01_Male") (at 353.06 71.12 180) (unit 1)
     (in_bom yes) (on_board yes)
-    (property "Reference" "J?" (id 0) (at 353.695 66.04 0))
+    (property "Reference" "J3" (id 0) (at 353.695 66.04 0))
     (property "Value" "Conn_01x01_Male" (id 1) (at 352.425 68.58 0))
     (property "Footprint" "Connector_PinHeader_1.00mm:PinHeader_1x01_P1.00mm_Vertical" (id 2) (at 353.06 71.12 0)
